Commit message: 将urdf文件生成xml文件，添加关节位置驱动器和关节阻尼和惯量，添加背景

File: rm_control/assets/overseas_65_b_v_description/.catkin_tools/realman_mujoco.urdf (robot description, URDF)
Before this commit: robot overseas_65_b_v_description, 33 links, 32 joints
Links:
- link base_link_underpan: geometry collision mesh filename=base_link_underpan.STL; visual mesh filename=base_link_underpan.STL
- link body_base_link: geometry collision mesh filename=body_base_link.STL; visual mesh filename=body_base_link.STL
- link camera_link: geometry collision mesh filename=camera_link.STL; visual mesh filename=camera_link.STL
- link head_link1: geometry collision mesh filename=head_link1.STL; visual mesh filename=head_link1.STL
- link head_link2: geometry collision mesh filename=head_link2.STL; visual mesh filename=head_link2.STL
- link l_base_link1: geometry collision mesh filename=l_base_link1.STL; visual mesh filename=l_base_link1.STL
- link l_hand_base_link: geometry collision mesh filename=l_hand_base_link.STL; visual mesh filename=l_hand_base_link.STL
- link l_link1: geometry collision mesh filename=l_link1.STL; visual mesh filename=l_link1.STL
- link l_link2: geometry collision mesh filename=l_link2.STL; visual mesh filename=l_link2.STL
- link l_link3: geometry collision mesh filename=l_link3.STL; visual mesh filename=l_link3.STL
- link l_link4: geometry collision mesh filename=l_link4.STL; visual mesh filename=l_link4.STL
- link l_link5: geometry collision mesh filename=l_link5.STL; visual mesh filename=l_link5.STL
- link l_link6: geometry collision mesh filename=l_link6.STL; visual mesh filename=l_link6.STL
- link link_left_wheel: geometry collision mesh filename=link_left_wheel.STL; visual mesh filename=link_left_wheel.STL
- link link_right_wheel: geometry collision mesh filename=link_right_wheel.STL; visual mesh filename=link_right_wheel.STL
- link link_swivel_wheel_1_1: geometry collision mesh filename=link_swivel_wheel_1_1.STL; visual mesh filename=link_swivel_wheel_1_1.STL
- link link_swivel_wheel_1_2: geometry collision mesh filename=link_swivel_wheel_1_2.STL; visual mesh filename=link_swivel_wheel_1_2.STL
- link link_swivel_wheel_2_1: geometry collision mesh filename=link_swivel_wheel_2_1.STL; visual mesh filename=link_swivel_wheel_2_1.STL
- link link_swivel_wheel_2_2: geometry collision mesh filename=link_swivel_wheel_2_2.STL; visual mesh filename=link_swivel_wheel_2_2.STL
- link link_swivel_wheel_3_1: geometry collision mesh filename=link_swivel_wheel_3_1.STL; visual mesh filename=link_swivel_wheel_3_1.STL
- link link_swivel_wheel_3_2: geometry collision mesh filename=link_swivel_wheel_3_2.STL; visual mesh filename=link_swivel_wheel_3_2.STL
- link link_swivel_wheel_4_1: geometry collision mesh filename=link_swivel_wheel_4_1.STL; visual mesh filename=link_swivel_wheel_4_1.STL
- link link_swivel_wheel_4_2: geometry collision mesh filename=link_swivel_wheel_4_2.STL; visual mesh filename=link_swivel_wheel_4_2.STL
- link platform_base_link: geometry collision mesh filename=platform_base_link.STL; visual mesh filename=platform_base_link.STL
- link r_base_link1: geometry collision mesh filename=r_base_link1.STL; visual mesh filename=r_base_link1.STL
- link r_hand_base_link: geometry collision mesh filename=r_hand_base_link.STL; visual mesh filename=r_hand_base_link.STL
- link r_link1: geometry collision mesh filename=r_link1.STL; visual mesh filename=r_link1.STL
- link r_link2: geometry collision mesh filename=r_link2.STL; visual mesh filename=r_link2.STL
- link r_link3: geometry collision mesh filename=r_link3.STL; visual mesh filename=r_link3.STL
- link r_link4: geometry collision mesh filename=r_link4.STL; visual mesh filename=r_link4.STL
- link r_link5: geometry collision mesh filename=r_link5.STL; visual mesh filename=r_link5.STL
- link r_link6: geometry collision mesh filename=r_link6.STL; visual mesh filename=r_link6.STL
